Commit message: January updates; start navigation

File: moony_description/robot/robot_gazebo.urdf1.xacro (robot description, xacro)
@@ -1,5 +1,5 @@
 <?xml version="1.0"?>
 <robot xmlns:xacro="http://www.ros.org/wiki/xacro" name="moony">
-<!-- <xacro:include filename="$(find moony_gazebo)/gazebo/diff_drive_gazebo.xacro" /> -->
+<!-- this robot can only go fwd and bwd, no turning -->
 <gazebo>
     <plugin name="gazebo_ros_control" filename="libgazebo_ros_control.so">
@@ -16,5 +16,5 @@
 <!-- for XACRO math - SPACES matter -->
 <xacro:property name="wheel_z" value="${-0.02 - base_height/2}" />
-<xacro:property name="wheel_r" value="${radians(90)}" />
+<xacro:property name="wheel_r" value="0" /> <!-- ${radians(90)}-->
 <xacro:property name="wheel_p" value="0" />
 <xacro:property name="wheel_y" value="0" />
@@ -24,5 +24,6 @@
 <xacro:property name="wheel_collision_radius" value="0.17" />
 <xacro:property name="wheel_collision_length" value="0.09" />
-<xacro:property name="wheel_mesh" value="package://moony_description/models/meshes/wheel.dae" />
+<xacro:property name="right" value="package://moony_description/models/meshes/wheel_left.dae" /> <!-- weird file name changing didn't do anything  -->
+<xacro:property name="left" value="package://moony_description/models/meshes/wheel_right.dae" />
 <xacro:property name="wheel_effort" value="0.1" />
 <xacro:property name="wheel_velocity" value="1" />
@@ -32,12 +33,7 @@
 <xacro:property name="wheel_dynamic_friction_coeff" value="10" />
 <!-- IMPORTS -->
-<!-- Import all Gazebo-customization elements, including Gazebo colors -->
-  <!-- <xacro:include filename="$(find moony_description)/robot/sensors.xacro" /> -->
-  <!-- THIS DID NOT WORK - you need to have the additional xacro with the proper headers: xml version and robot declaration -->
-  <!-- Import Rviz colors -->
-  <!-- <xacro:include filename="$(find rrbot_description)/urdf/materials.xacro" /> -->
 <!-- MACROS -->
-<xacro:macro name="individual_wheel" params="num x y r">
-   <link name="wheel_${num}_link">
+<xacro:macro name="individual_wheel_left" params="depth x y">
+   <link name="wheel_${depth}_left_link">
         <inertial>
             <origin rpy="0 0 0" xyz="0 0 0"/>
@@ -48,5 +44,5 @@
         </inertial>
         <collision>
-            <origin rpy="0 0 0" xyz="0 0 0"/> <!-- pre joint orientation -->
+            <origin rpy="${radians(90)} 0 0" xyz="0 0 0"/> <!-- pre joint orientation -->
             <geometry>
                 <cylinder radius="${wheel_collision_radius}" length="${wheel_collision_length}"/>
@@ -56,29 +52,77 @@
             <origin rpy="0 0 0" xyz="0 0 0"/> <!-- center of the wheel -->
             <geometry>
-                <mesh filename="${wheel_mesh}"/>
+                <mesh filename="${left}"/>
             </geometry>
             <!-- <material name="white"/> only used in rviz for simple geometry -->
         </visual>
     </link>
-        <gazebo reference="wheel_${num}_link">
+        <gazebo reference="wheel_${depth}_left_link">
             <kp>100000.0</kp>   <!-- kp: This coefficient sets the static contact stiffness -->
             <kd>100000.0</kd>   <!-- kd: This coefficient sets the dynamic contact stiffness -->
             <mu1>10.0</mu1>     <!-- mu1: The static friction coefficient -->
             <mu2>10.0</mu2>     <!-- mu2: The dynamic friction coefficient. -->
-            <!-- <material>Gazebo/Yellow</material> -->
+            <material>Gazebo/Yellow</material>
         </gazebo>
-    <joint name="wheel_${num}_joint" type="continuous">
-        <parent link="base_link"/>
-        <child link="wheel_${num}_link"/>
-        <origin xyz="${x} ${y} ${wheel_z}" rpy="${r} ${wheel_p} ${wheel_y}"/> <!-- joint location -->
+    <joint name="wheel_${depth}_left_joint" type="continuous">
+        <parent link="base_link"/>
+        <child link="wheel_${depth}_left_link"/>
+        <origin xyz="${x} ${y} ${wheel_z}" rpy="${wheel_r} ${wheel_p} ${wheel_y}"/> <!-- joint location -->
         <limit effort="${wheel_effort}" velocity="${wheel_velocity}"/>
-        <axis xyz="0 0 1"/>
-    </joint>
-    <transmission name="wheel_tran_${num}">
+        <axis xyz="0 1 0"/>
+    </joint>
+    <transmission name="wheel_tran_${depth}_left">
         <type>transmission_interface/SimpleTransmission</type>
-        <joint name="wheel_${num}_joint">
+        <joint name="wheel_${depth}_left_joint">
             <hardwareInterface>hardware_interface/VelocityJointInterface</hardwareInterface>
         </joint>
-        <actuator name="wheel_motor_${num}">
+        <actuator name="wheel_motor_${depth}_left">
+            <hardwareInterface>VelocityJointInterface</hardwareInterface>
+            <mechanicalReduction>1</mechanicalReduction>
+        </actuator>
+    </transmission>
+</xacro:macro>
+<xacro:macro name="individual_wheel_right" params="depth x y">
+   <link name="wheel_${depth}_right_link">
+        <inertial>
+            <origin rpy="0 0 0" xyz="0 0 0"/>
+            <mass value="${wheel_mass}" />
+            <inertia ixx="${wheel_inertia_ixx}" ixy="0" ixz="0" iyy="${wheel_inertia_iyy}" iyz="0" izz="${wheel_inertia_izz}"/>
+             <!-- values taken from solidworks; the origin is the position of the part
+                w.r.t its axes for the second moment of mass values  -->
+        </inertial>
+        <collision>
+            <origin rpy="${radians(90)} 0 0" xyz="0 0 0"/> <!-- pre joint orientation -->
+            <geometry>
+                <cylinder radius="${wheel_collision_radius}" length="${wheel_collision_length}"/>
+            </geometry>
+        </collision>
+        <visual>
+            <origin rpy="0 0 0" xyz="0 0 0"/> <!-- center of the wheel -->
+            <geometry>
+                <mesh filename="${right}"/>
+            </geometry>
+            <!-- <material name="white"/> only used in rviz for simple geometry -->
+        </visual>
+    </link>
+        <gazebo reference="wheel_${depth}_right_link">
+            <kp>100000.0</kp>   <!-- kp: This coefficient sets the static contact stiffness -->
+            <kd>100000.0</kd>   <!-- kd: This coefficient sets the dynamic contact stiffness -->
+            <mu1>10.0</mu1>     <!-- mu1: The static friction coefficient -->
+            <mu2>10.0</mu2>     <!-- mu2: The dynamic friction coefficient. -->
+            <material>Gazebo/Yellow</material>
+        </gazebo>
+    <joint name="wheel_${depth}_right_joint" type="continuous">
+        <parent link="base_link"/>
+        <child link="wheel_${depth}_right_link"/>
+        <origin xyz="${x} ${y} ${wheel_z}" rpy="${wheel_r} ${wheel_p} ${wheel_y}"/> <!-- joint location -->
+        <limit effort="${wheel_effort}" velocity="${wheel_velocity}"/>
+        <axis xyz="0 1 0"/>
+    </joint>
+    <transmission name="wheel_tran_${depth}_right">
+        <type>transmission_interface/SimpleTransmission</type>
+        <joint name="wheel_${depth}_right_joint">
+            <hardwareInterface>hardware_interface/VelocityJointInterface</hardwareInterface>
+        </joint>
+        <actuator name="wheel_motor_${depth}_right">
             <hardwareInterface>VelocityJointInterface</hardwareInterface>
             <mechanicalReduction>1</mechanicalReduction>
@@ -120,9 +164,9 @@
         </visual>
     </link>
-   <xacro:individual_wheel num="1" x="${1.0 * wheel_x}" y="${1.0 * .24}" r="${-1 * wheel_r}"/>
-   <xacro:individual_wheel num="2" x="${-1.0 * wheel_x}" y="${1.0 * .24}" r="${-1 * wheel_r}"/>
-   <xacro:individual_wheel num="3" x="${1.0 * wheel_x}" y="${-1.0 * .24}" r="${1 * wheel_r}"/>
-   <xacro:individual_wheel num="4" x="${-1.0 * wheel_x}" y="${-1.0 * .24}" r="${1 * wheel_r}"/>
-   <!-- <xacro:individual_wheel num="1" x="0" y="0" r="${-1 * wheel_r}"/> -->
+   <xacro:individual_wheel_left depth="front" x="${1.0 * wheel_x}" y="${1.0 * .24}" />
+   <xacro:individual_wheel_left depth="rear" x="${-1.0 * wheel_x}" y="${1.0 * .24}" />
+   <xacro:individual_wheel_right depth="front" x="${1.0 * wheel_x}" y="${-1.0 * .24}"/>
+   <xacro:individual_wheel_right depth="rear" x="${-1.0 * wheel_x}" y="${-1.0 * .24}"/>
+<!-- <xacro:include filename="$(find moony_gazebo)/gazebo/diff_drive_gazebo.xacro" /> -->
    <!-- <xacro:differential_drive prefix="front" left="1" right="3"/> -->
    <!-- <xacro:differential_drive prefix="back" left="2" right="4"/> -->

File: moony_description/robot/robot_skid.xacro (robot description, xacro)
@@ -1,92 +1,25 @@
 <?xml version="1.0"?>
 <robot xmlns:xacro="http://www.ros.org/wiki/xacro" name="moony">
-<xacro:include filename="$(find moony_gazebo)/gazebo/sensors.xacro" />
+<!-- note: units are meters, kilograms, and radians -->
+<!-- THIS PLUGIN NEEDS TO BE FIRST -->
+<gazebo>
+    <plugin name="gazebo_ros_control" filename="libgazebo_ros_control.so">
+        <robotNamespace>/moony</robotNamespace>
+    </plugin>
+</gazebo>
 <!-- CONSTANTS -->
 <xacro:property name="base_mass" value="4.11" />
 <xacro:property name="base_height" value=".03" />
-<xacro:property name="wheel_mass" value="2" />
-<xacro:property name="wheel_x" value="0.3" />
-<xacro:property name="wheel_y" value="${(.38/2)+.04+.01}" />
-<!-- y = width/2 of frame + wheel COG to wall + buffer -->
-<!-- for XACRO math - SPACES matter -->
-<xacro:property name="wheel_z" value="${-0.02 - base_height/2}" />
-<xacro:property name="wheel_r" value="${radians(90)}" />
-<xacro:property name="wheel_p" value="0" />
-<xacro:property name="wheel_y" value="0" />
-<xacro:property name="wheel_inertia_ixx" value="0.02" />
-<xacro:property name="wheel_inertia_iyy" value="0.02" />
-<xacro:property name="wheel_inertia_izz" value="0.04" />
-<xacro:property name="wheel_collision_radius" value="0.17" />
-<xacro:property name="wheel_collision_length" value="0.09" />
-<xacro:property name="wheel_mesh" value="package://moony_description/models/meshes/wheel.dae" />
-<xacro:property name="wheel_effort" value="0.1" />
-<xacro:property name="wheel_velocity" value="1" />
-<xacro:property name="wheel_static_contact_stiffness" value="100000" />
-<xacro:property name="wheel_dynamic_contact_stiffness" value="100000" />
-<xacro:property name="wheel_static_friction_coeff" value="10" />
-<xacro:property name="wheel_dynamic_friction_coeff" value="10" />
 <!-- IMPORTS -->
-<!-- Import all Gazebo-customization elements, including Gazebo colors -->
-  <!-- <xacro:include filename="$(find moony_description)/robot/sensors.xacro" /> -->
-  <!-- THIS DID NOT WORK - you need to have the additional xacro with the proper headers: xml version and robot declaration -->
-  <!-- Import Rviz colors -->
-  <!-- <xacro:include filename="$(find rrbot_description)/urdf/materials.xacro" /> -->
-<!-- MACROS -->
-<xacro:macro name="individual_wheel" params="num x y r">
-   <link name="wheel_${num}_link">
-        <inertial>
-            <origin rpy="0 0 0" xyz="0 0 0"/>
-            <mass value="${wheel_mass}" />
-            <inertia ixx="${wheel_inertia_ixx}" ixy="0" ixz="0" iyy="${wheel_inertia_iyy}" iyz="0" izz="${wheel_inertia_izz}"/>
-             <!-- values taken from solidworks; the origin is the position of the part
-                w.r.t its axes for the second moment of mass values  -->
-        </inertial>
-        <collision>
-            <origin rpy="0 0 0" xyz="0 0 0"/> <!-- pre joint orientation -->
-            <geometry>
-                <cylinder radius="${wheel_collision_radius}" length="${wheel_collision_length}"/>
-            </geometry>
-        </collision>
-        <visual>
-            <origin rpy="0 0 0" xyz="0 0 0"/> <!-- center of the wheel -->
-            <geometry>
-                <mesh filename="${wheel_mesh}"/>
-            </geometry>
-            <!-- <material name="white"/> only used in rviz for simple geometry -->
-        </visual>
-    </link>
-        <gazebo reference="wheel_${num}_link">
-            <kp>100000.0</kp>   <!-- kp: This coefficient sets the static contact stiffness -->
-            <kd>100000.0</kd>   <!-- kd: This coefficient sets the dynamic contact stiffness -->
-            <mu1>10.0</mu1>     <!-- mu1: The static friction coefficient -->
-            <mu2>10.0</mu2>     <!-- mu2: The dynamic friction coefficient. -->
-            <!-- <material>Gazebo/Yellow</material> -->
-        </gazebo>
-    <joint name="wheel_${num}_joint" type="continuous">
-        <parent link="base_link"/>
-        <child link="wheel_${num}_link"/>
-        <origin xyz="${x} ${y} ${wheel_z}" rpy="${r} ${wheel_p} ${wheel_y}"/> <!-- joint location -->
-        <limit effort="${wheel_effort}" velocity="${wheel_velocity}"/>
-        <axis xyz="0 0 1"/>
-    </joint>
-    <transmission name="wheel_tran_${num}">
-        <type>transmission_interface/SimpleTransmission</type>
-        <joint name="wheel_${num}_joint">
-            <hardwareInterface>hardware_interface/VelocityJointInterface</hardwareInterface>
-        </joint>
-        <actuator name="wheel_motor_${num}">
-            <hardwareInterface>VelocityJointInterface</hardwareInterface>
-            <mechanicalReduction>1</mechanicalReduction>
-        </actuator>
-    </transmission>
-</xacro:macro>
-<!-- note: units are meters, kilograms, and radians -->
-    <link name="base_footprint" />
+<xacro:include filename="$(find moony_gazebo)/gazebo/sensors.xacro" />
+<xacro:include filename="$(find moony_gazebo)/gazebo/macros.xacro" />
+<xacro:include filename="$(find moony_gazebo)/gazebo/skid_drive.xacro" />
+<!-- LINKS -->
+    <link name="base_footprint" /> <!-- dummy prevents laser from publishing -->
     <joint name="base_joint" type="fixed">
-     <origin xyz="0 0 .1" rpy="0 0 0" />
+     <origin xyz="0 0 0" rpy="0 0 0" />
      <parent link="base_footprint"/>
      <child link="base_link"/>
    </joint>
-        <!-- dummy prevents laser from publishing -->
     <link name="base_link">
         <inertial>
@@ -110,11 +43,8 @@
         </visual>
     </link>
-   <xacro:individual_wheel num="1" x="${1.0 * wheel_x}" y="${1.0 * .24}" r="${-1 * wheel_r}"/>
-   <xacro:individual_wheel num="2" x="${-1.0 * wheel_x}" y="${1.0 * .24}" r="${-1 * wheel_r}"/>
-   <xacro:individual_wheel num="3" x="${1.0 * wheel_x}" y="${-1.0 * .24}" r="${1 * wheel_r}"/>
-   <xacro:individual_wheel num="4" x="${-1.0 * wheel_x}" y="${-1.0 * .24}" r="${1 * wheel_r}"/>
-   <!-- <xacro:individual_wheel num="1" x="0" y="0" r="${-1 * wheel_r}"/> -->
-   <!-- <xacro:differential_drive prefix="front" left="1" right="3"/> -->
-   <!-- <xacro:differential_drive prefix="back" left="2" right="4"/> -->
+   <xacro:individual_wheel num="1" x="1.0" y="1.0" r="-1.0"/>
+   <xacro:individual_wheel num="2" x="-1.0" y="1.0" r="-1.0"/>
+   <xacro:individual_wheel num="3" x="1.0" y="-1.0" r="1.0"/>
+   <xacro:individual_wheel num="4" x="-1.0" y="-1.0" r="1.0"/>
      <!-- Lidar Link -->
   <link name="lidar_link">

File: moony_description/urdf/robot_gazebo_simple.urdf (robot description, URDF)
Before this commit: robot first_robot, 2 links, 1 joints
Links:
- link wheel_1_link: geometry collision cylinder length=0.03125 radius=0.125; visual mesh filename=package://moony_description/models/meshes/wheel_left.dae

File: moony_gazebo/gazebo/sensors.xacro (robot description, xacro)
@@ -1,9 +1,4 @@
 <?xml version="1.0"?>
 <robot xmlns:xacro="http://www.ros.org/wiki/xacro" name="moony">
-<gazebo>
-    <plugin name="gazebo_ros_control" filename="libgazebo_ros_control.so">
-        <robotNamespace>/moony</robotNamespace>
-    </plugin>
-</gazebo>
 <gazebo reference="lidar_link">
        <kp>100000.0</kp>   <!-- kp: This coefficient sets the static contact stiffness -->

File: moony_gazebo/gazebo/skid_drive.xacro (robot description, xacro)
@@ -4,15 +4,21 @@
   <plugin name="skid_steer_drive_controller" filename="libgazebo_ros_skid_steer_drive.so">
     <updateRate>100.0</updateRate>
-    <robotNamespace>/</robotNamespace>
-    <leftFrontJoint>front_left_wheel_joint</leftFrontJoint>
-    <rightFrontJoint>front_right_wheel_joint</rightFrontJoint>
-    <leftRearJoint>back_left_wheel_joint</leftRearJoint>
-    <rightRearJoint>back_right_wheel_joint</rightRearJoint>
-    <wheelSeparation>0.4</wheelSeparation>
-    <wheelDiameter>0.215</wheelDiameter>
+    <robotNamespace>/moony</robotNamespace>
+    <leftFrontJoint>wheel_1_joint</leftFrontJoint>
+    <rightFrontJoint>wheel_3_joint</rightFrontJoint>
+    <leftRearJoint>wheel_2_joint</leftRearJoint>
+    <rightRearJoint>wheel_4_joint</rightRearJoint>
+    <wheelSeparation>${wheel_y * 2}</wheelSeparation>
+    <wheelDiameter>${wheel_collision_radius}</wheelDiameter>
     <robotBaseFrame>base_link</robotBaseFrame>
+    <topicName>/moony/cmd_vel</topicName>
+    <commandTopic>/moony/cmd_vel</commandTopic>
     <torque>20</torque>
-    <topicName>cmd_vel</topicName>
+    <odometryTopic>odom</odometryTopic>
+    <odometryFrame>odom</odometryFrame>
     <broadcastTF>false</broadcastTF>
+    <covariance_x>0.000100</covariance_x>
+    <covariance_y>0.000100</covariance_y>
+    <covariance_yaw>0.010000</covariance_yaw>
   </plugin>
 </gazebo>
