Commit message: cleaned up moony_gazebo launch

File: moony_description/robot/robot_skid.xacro (robot description, xacro)
@@ -16,11 +16,11 @@
 <xacro:include filename="$(find moony_gazebo)/gazebo/skid_drive.xacro" />
 <!-- LINKS -->
-    <link name="base_footprint" /> <!-- dummy prevents laser from publishing -->
+    <link name="base_link" /> <!-- dummy prevents laser from publishing -->
     <joint name="base_joint" type="fixed">
-     <origin xyz="0 0 0" rpy="0 0 0" />
-     <parent link="base_footprint"/>
-     <child link="base_link"/>
+     <origin xyz="0 0 0.01" rpy="0 0 0" />
+     <parent link="base_link"/>
+     <child link="body_link"/>
    </joint>
-    <link name="base_link">
+    <link name="body_link">
         <inertial>
             <origin rpy="0 0 0" xyz="0 0 0"/>
@@ -73,5 +73,5 @@
   </link>
     <joint name="lidar_joint" type="fixed">
-        <parent link="base_link"/>
+        <parent link="body_link"/>
         <child link="lidar_link"/>
         <origin xyz=".47 0 ${-0.015 - 0.005/2 -0.001}" rpy="${radians(180)} 0 0"/> <!-- joint location -->
@@ -102,5 +102,5 @@
   </link>
     <joint name="imu_joint" type="fixed">
-        <parent link="base_link"/>
+        <parent link="body_link"/>
         <child link="imu_link"/>
         <origin xyz="0 0.17 ${+0.015 + 0.005/2 +0.001}" rpy="0 0 0"/> <!-- joint location -->

File: moony_gazebo/gazebo/macros.xacro (robot description, xacro)
@@ -39,5 +39,5 @@
         </gazebo>
     <joint name="wheel_${num}_joint" type="continuous">
-        <parent link="base_link"/>
+        <parent link="body_link"/>
         <child link="wheel_${num}_link"/>
         <origin xyz="${x * 0.3} ${y * wheel_y} ${-0.02 - base_height/2}" rpy="0 0 0"/> <!-- joint location -->

File: moony_gazebo/gazebo/sensors.xacro (robot description, xacro)
@@ -2,10 +2,7 @@
 <robot xmlns:xacro="http://www.ros.org/wiki/xacro" name="moony">
 <gazebo reference="lidar_link">
-       <kp>100000.0</kp>   <!-- kp: This coefficient sets the static contact stiffness -->
-        <kd>100000.0</kd>   <!-- kd: This coefficient sets the dynamic contact stiffness -->
-        <mu1>10.0</mu1>     <!-- mu1: The static friction coefficient -->
-        <mu2>10.0</mu2>     <!-- mu2: The dynamic friction coefficient. -->
+<!-- do not need kd, kp, mu1, and mu2 -->
     <sensor type="ray" name="front_rplidar_sensor">
-      <pose>0 0 0 0 0 0</pose>
+      <pose>0 0 0.04 0 0 0</pose>
       <visualize>true</visualize>
       <update_rate>40</update_rate>
@@ -13,5 +10,5 @@
         <scan>
           <horizontal>
-            <samples>720</samples>
+            <samples>9200</samples>
             <resolution>1</resolution>
             <min_angle>${-radians(360)}</min_angle>
@@ -22,5 +19,5 @@
           <min>0.10</min>
           <max>30.0</max>
-          <resolution>0.01</resolution>
+          <resolution>0.03</resolution>
         </range>
         <noise>
@@ -31,5 +28,5 @@
                reading. -->
           <mean>0.0</mean>
-          <stddev>0.01</stddev>
+          <stddev>0.001</stddev>
         </noise>
       </ray>
@@ -47,9 +44,9 @@
       <update_rate>100</update_rate>
       <visualize>true</visualize>
-      <topic>__default_topic__</topic>
+      <topic>/moony/imu</topic>
       <plugin filename="libgazebo_ros_imu_sensor.so" name="imu_plugin">
         <topicName>/moony/imu</topicName>
         <bodyName>imu_link</bodyName>
-        <updateRateHZ>10.0</updateRateHZ>
+        <updateRateHZ>100.0</updateRateHZ>
         <gaussianNoise>0.0</gaussianNoise>
         <xyzOffset>0 0 0</xyzOffset>

File: moony_gazebo/gazebo/skid_drive.xacro (robot description, xacro)
@@ -15,6 +15,6 @@
     <commandTopic>/moony/cmd_vel</commandTopic>
     <torque>20</torque>
-    <odometryTopic>/moony/odom</odometryTopic>
-    <odometryFrame>imu_link</odometryFrame>
+    <odometryTopic>notUsed</odometryTopic>
+    <odometryFrame>notUsed</odometryFrame>
     <broadcastTF>false</broadcastTF>
     <covariance_x>0.000100</covariance_x>

Commit message: working on gmapping bug

File: moony_description/robot/robot_skid.xacro (robot description, xacro)
@@ -13,14 +13,14 @@
 <!-- IMPORTS -->
 <xacro:include filename="$(find moony_gazebo)/gazebo/sensors.xacro" />
-<xacro:include filename="$(find moony_gazebo)/gazebo/macros.xacro" />
+<xacro:include filename="$(find moony_gazebo)/gazebo/wheels.xacro" />
 <xacro:include filename="$(find moony_gazebo)/gazebo/skid_drive.xacro" />
 <!-- LINKS -->
-    <link name="base_link" /> <!-- dummy prevents laser from publishing -->
+    <link name="base_footprint" /> <!-- dummy prevents laser from publishing -->
     <joint name="base_joint" type="fixed">
      <origin xyz="0 0 0.01" rpy="0 0 0" />
-     <parent link="base_link"/>
-     <child link="body_link"/>
+     <parent link="base_footprint"/>
+     <child link="base_link"/>
    </joint>
-    <link name="body_link">
+    <link name="base_link">
         <inertial>
             <origin rpy="0 0 0" xyz="0 0 0"/>
@@ -73,9 +73,8 @@
   </link>
     <joint name="lidar_joint" type="fixed">
-        <parent link="body_link"/>
+        <parent link="base_link"/>
         <child link="lidar_link"/>
-        <origin xyz=".47 0 ${-0.015 - 0.005/2 -0.001}" rpy="${radians(180)} 0 0"/> <!-- joint location -->
+        <origin xyz=".47 0 ${-0.015 - 0.005/2 -0.001}" rpy="${radians(180)} 0 0"/> <!-- joint location - this may be the plane of the laser-->
     </joint>
-<!-- lidar sensor -->
 <!-- IMU sensor -->
  <link name="imu_link">
@@ -102,5 +101,5 @@
   </link>
     <joint name="imu_joint" type="fixed">
-        <parent link="body_link"/>
+        <parent link="base_link"/>
         <child link="imu_link"/>
         <origin xyz="0 0.17 ${+0.015 + 0.005/2 +0.001}" rpy="0 0 0"/> <!-- joint location -->

File: moony_gazebo/gazebo/skid_drive.xacro (robot description, xacro)
@@ -12,4 +12,5 @@
     <wheelDiameter>${wheel_collision_radius}</wheelDiameter>
     <robotBaseFrame>base_link</robotBaseFrame>
+    <!-- should this be base_footprint? -->
     <topicName>/moony/cmd_vel</topicName>
     <commandTopic>/moony/cmd_vel</commandTopic>

File: moony_gazebo/gazebo/wheels.xacro (robot description, xacro)
@@ -39,5 +39,5 @@
         </gazebo>
     <joint name="wheel_${num}_joint" type="continuous">
-        <parent link="body_link"/>
+        <parent link="base_link"/>
         <child link="wheel_${num}_link"/>
         <origin xyz="${x * 0.3} ${y * wheel_y} ${-0.02 - base_height/2}" rpy="0 0 0"/> <!-- joint location -->
