Commit message: implemented robot_localization, added cameras

File: moony_description/robot/Parts/mount_cameras.urdf.xacro (robot description, xacro)
@@ -6,5 +6,5 @@
             <origin xyz="0 0 ${.1/2}" rpy="0 0 0"/>
             <geometry>
-                <box size="0.2 0.1 0.1"/>
+                <box size="0.1 0.05 0.05"/>
             </geometry>
             </collision>
@@ -12,5 +12,5 @@
             <origin xyz="0 0 0" rpy="0 0 0"/>
             <geometry>
-                <box size="0.2 0.1 0.1"/>
+                <box size="0.1 0.05 0.05"/>
             </geometry>
             </visual>
@@ -27,5 +27,5 @@
             <parent link="base_link"/>
             <child link="${side}_camera_link"/>
-            <origin xyz="${x} ${y} ${+0.015 + 0.005/2 +0.001}" rpy="0 0 0"/> <!-- joint location -->
+            <origin xyz="${x} ${y} ${0.05}" rpy="0 0 0"/> <!-- joint location -->
         </joint>
     </xacro:macro>

File: moony_description/robot/robot_skid.urdf.xacro (robot description, xacro)
@@ -48,10 +48,11 @@
  <xacro:include filename="$(find moony_description)/robot/Parts/mount_lidar.urdf.xacro" />
  <xacro:include filename="$(find moony_description)/robot/Parts/mount_imu.urdf.xacro" />
- <xacro:include filename="$(find moony_description)/robot/Parts/mount_cameras.urdf.xacro" />
+ <!-- <xacro:include filename="$(find moony_description)/robot/Parts/mount_cameras.urdf.xacro" />
     <xacro:camera side="left" x="0.47" y="0.17" />
+    <xacro:camera side="right" x="0.47" y="-0.17" /> -->
 <!-- Include gazebo simulation parameters -->
 <xacro:include filename="$(find moony_gazebo)/gazebo/skid_drive.xacro" />
 <xacro:include filename="$(find moony_gazebo)/gazebo/sensors.xacro" />
-<xacro:include filename="$(find moony_gazebo)/gazebo/cameras.xacro" />
-    <xacro:camera_gazebo side="left" />
+<!-- <xacro:include filename="$(find moony_gazebo)/gazebo/cameras.xacro" /> -->
+    <!-- <xacro:camera_gazebo side="left" /> -->
 </robot>

File: moony_gazebo/gazebo/cameras.xacro (robot description, xacro)
@@ -2,5 +2,62 @@
 <robot xmlns:xacro="http://www.ros.org/wiki/xacro" name="moony">
  <xacro:macro name="camera_gazebo" params="side">
-  <gazebo reference="${side}_camera_link">
+<!-- MULTICAMERA - STEREO CAMERAS -->
+ <gazebo reference="${side}_camera_link">
+    <sensor type="multicamera" name="stereo_camera">
+      <update_rate>30.0</update_rate>
+      <camera name="left">
+        <horizontal_fov>1.3962634</horizontal_fov>
+        <image>
+          <width>800</width>
+          <height>800</height>
+          <format>R8G8B8</format>
+        </image>
+        <clip>
+          <near>0.02</near>
+          <far>300</far>
+        </clip>
+        <noise>
+          <type>gaussian</type>
+          <mean>0.0</mean>
+          <stddev>0.007</stddev>
+        </noise>
+      </camera>
+      <camera name="right">
+        <pose>0 ${-0.17*2} 0 0 0 0</pose>
+        <horizontal_fov>1.3962634</horizontal_fov>
+        <image>
+          <width>800</width>
+          <height>800</height>
+          <format>R8G8B8</format>
+        </image>
+        <clip>
+          <near>0.02</near>
+          <far>300</far>
+        </clip>
+        <noise>
+          <type>gaussian</type>
+          <mean>0.0</mean>
+          <stddev>0.007</stddev>
+        </noise>
+      </camera>
+      <plugin name="stereo_camera_controller" filename="libgazebo_ros_multicamera.so">
+        <alwaysOn>true</alwaysOn>
+        <updateRate>0.0</updateRate>
+        <cameraName>moony/${side}_camera</cameraName>
+        <imageTopicName>image_raw</imageTopicName>
+        <cameraInfoTopicName>camera_info</cameraInfoTopicName>
+        <frameName>${side}_camera_link</frameName>
+        <!--<rightFrameName>right_camera_optical_frame</rightFrameName>-->
+        <hackBaseline>0.07</hackBaseline>
+        <distortionK1>0.0</distortionK1>
+        <distortionK2>0.0</distortionK2>
+        <distortionK3>0.0</distortionK3>
+        <distortionT1>0.0</distortionT1>
+        <distortionT2>0.0</distortionT2>
+      </plugin>
+    </sensor>
+  </gazebo>
+ <!-- SINGLE CAMERA -->
+  <!-- <gazebo reference="${side}_camera_link">
     <sensor type="camera" name="${side}_camera">
       <update_rate>30.0</update_rate>
@@ -17,9 +74,9 @@
         </clip>
         <noise>
-          <type>gaussian</type>
+          <type>gaussian</type> -->
           <!-- Noise is sampled independently per pixel on each frame.
                That pixel's noise value is added to each of its color
                channels, which at that point lie in the range [0,1]. -->
-          <mean>0.0</mean>
+    <!--      <mean>0.0</mean>
           <stddev>0.007</stddev>
         </noise>
@@ -40,5 +97,5 @@
       </plugin>
     </sensor>
-  </gazebo>
+  </gazebo> -->
   </xacro:macro>
 </robot>

File: moony_gazebo/gazebo/skid_drive.xacro (robot description, xacro)
@@ -18,5 +18,5 @@
     <odometryTopic>skid_drive</odometryTopic>
     <odometryFrame>skid_drive</odometryFrame>
-    <broadcastTF>false</broadcastTF>
+    <broadcastTF>true</broadcastTF> <!-- made this true for the robot_localization package; ODOM -> BASE LINK -->
     <covariance_x>0.000100</covariance_x>
     <covariance_y>0.000100</covariance_y>
