Commit message: physical testing. beacons work. next - calibrating the imu to remove its bias

File: moony_description/robot/Parts/real_beacon.urdf.xacro (robot description, xacro)
@@ -25,7 +25,7 @@
   </link>
     <joint name="beacon_joint" type="fixed">
-        <parent link="controls_box"/>
+        <parent link="base_link"/>
         <child link="beacon_link"/>
-        <origin xyz="${0.09/2} ${0.38/2} ${z/2 + 0.2985/2}" rpy="0 0 0"/> <!-- joint location -->
+        <origin xyz="${-0.47} ${0.0} ${z/2 + 0.01}" rpy="0 0 0"/> <!-- joint location -->
     </joint>
 </robot>

Commit message: one beacon working

File: moony_description/robot/Parts/real_beacon.urdf.xacro (robot description, xacro)
@@ -1,10 +1,12 @@
 <?xml version="1.0"?>
 <robot xmlns:xacro="http://www.ros.org/wiki/xacro" name="moony">
-<xacro:property name="z" value="${0.125}" />
+<xacro:property name="z" value="${0.0938}" />
+<xacro:property name="y" value="${0.0485}" />
+<xacro:property name="x" value="${0.015}" />
  <link name="beacon_link">
     <collision>
-      <origin xyz="0 0 ${.05/2}" rpy="0 0 0"/>
+      <origin xyz="0 0 0" rpy="0 0 0"/>
       <geometry>
-        <box size="0.05 0.05 ${z}"/>
+        <box size="${x} ${y} ${z}"/>
       </geometry>
     </collision>
@@ -12,5 +14,5 @@
       <origin xyz="0 0 0" rpy="0 0 0"/>
       <geometry>
-        <box size="0.025 0.025 0.075"/>
+        <box size="${x} ${y} ${z}"/>
       </geometry>
     </visual>
@@ -27,5 +29,5 @@
         <parent link="base_link"/>
         <child link="beacon_link"/>
-        <origin xyz="${-0.47} ${0.0} ${z/2 + 0.01}" rpy="0 0 0"/> <!-- joint location -->
+        <origin xyz="${-0.49} ${0.165} ${z/2 +0.0125}" rpy="0 0 3.141592653589793"/> <!-- joint location -->
     </joint>
 </robot>

File: moony_description/robot/Parts/real_imu.urdf.xacro (robot description, xacro)
@@ -28,3 +28,4 @@
         <origin xyz="0.47 0.15 -${+0.015 + 0.005/2}" rpy="0 3.141592653589793 1.5707963267948966"/> <!-- joint location -->
     </joint>
+    <!-- rpy="0 3.141592653589793 1.5707963267948966" upside down, y direction in forward orientation, z down-->
 </robot>
